File: Adapters/LVDSAdapterBoard/LVDSAdapterBoard.kicad_pcb (KiCad board)
At the start: 2 copper layers, 33.2 x 18.2 mm, 5 parts, among them J1 Main Board Connector, J2 LCD Connector Top, J3 LCD Connector Bottom

Commit message: KiCad version update
Other:
- net class Default removed
