File: Adapters/LVDSAdapterBoardSingle/LVDSAdapterBoardSingle.kicad_pcb (KiCad board)
At the start: 2 copper layers, 33.2 x 18.2 mm, 4 parts, among them J1 Main Board Connector, J3 LCD Connector Bottom

Commit message: KiCad version update
Other:
- net class Default removed
