File: RTD2662Board.kicad_pcb (KiCad board)
At the start: 2 copper layers, 100 x 70 mm, 260 parts, among them J1 DVI, J10 UART/I2C, J11 LCD Connector, J12 SPDIFF, J13 3.5mm jack, J14 DC Jack, J15 Expansion Connector, J2 HDMI A, J3 3.5mm jack, J4 VGA, J5 CVBS1, J6 CVBS2, J7 Mini-DIN-4, J8 USB B, J9 Keyboard Connector, Q1 BC846, Q2 BC846, Q3 AO3401A, Q4 BC846, Q5 AO3401A, SW1 POWER, SW2 MENU, SW3 UP, SW4 DOWN, SW5 SOURCE, U1 RTD2662, U10 25x128, U11 APW7313, U12 AMS1117-1.8, U2 TPS61040DBV, U3 TL1838, U4 CH341T, U5 TPS61040DBV, U6 ES7134S, U7 PAM8003, U8 TPS61040DBV, U9 24x01, Y1 27MHz, Y2 12MHz

Commit message: Replace U5, TPS61040DBV with PT4103 (White LED Step-Up Converter).
Parts:
- U5: value TPS61040DBV -> PT4103; footprint Package_TO_SOT_SMD:SOT-23-5 -> Package_TO_SOT_SMD:SOT-23-6
- U7: footprint Package_SO:SO-16_3.9x9.9mm_P1.27mm -> RTD2662Board:HSOP-16-1EP_3.9x9.9mm_P1.27mm_EP2.41x4.1mm
Connections:
- U5 pad 5: +3V3 -> BL_ANO
- U7 pad 10: Net-(R63-Pad1) -> Net-(U7-RIN)
- U7 pad 12: Net-(C52-Pad1) -> Net-(U7-VOL)
- U7 pad 6: Net-(C50-Pad1) -> Net-(U7-VREF)
- U7 pad 7: Net-(R61-Pad1) -> Net-(U7-LIN)
Routing:
- net GND: track 244.7 -> 256.4 mm
- net Net-(U7-LIN): track 0.00 -> 9.01 mm, vias 0 -> 2
- net Net-(R61-Pad1): track 9.01 -> 0.00 mm, vias 2 -> 0
- net Net-(U7-VOL): track 0.00 -> 5.61 mm
- net Net-(C52-Pad1): track 4.89 -> 0.00 mm
- net BL_ANO: track 16.1 -> 20.8 mm, vias 2 -> 3
- net Net-(U7-RIN): track 0.00 -> 3.20 mm
- net Net-(R63-Pad1): track 3.20 -> 0.00 mm
- net Net-(U7-VREF): track 0.00 -> 2.20 mm
- net Net-(C50-Pad1): track 2.20 -> 0.00 mm
- net BL_CAT: track 18.1 -> 18.9 mm

Commit message: Correct resistor value, replace connector values
Parts:
- J5: value CVBS1 -> RCA Jack
- J6: value CVBS2 -> CVBS
- R58: value 6.8Ω -> 0.68Ω
Routing:
- net GND: track 256.4 -> 261.0 mm
Changed lines of the file:
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@@
         (effects (font (size 1.001402 1.001402) (thickness 0.15)))
     )
-    (fp_text value "CVBS1" (at 0.065075 5.499085 180) (layer "F.Fab")
+    (fp_text value "RCA Jack" (at 0.065075 5.499085 180) (layer "F.Fab")
         (effects (font (size 1.000748 1.000748) (thickness 0.15)))
     )
@@
         (effects (font (size 1 1) (thickness 0.15)))
     )
-    (fp_text value "CVBS2" (at 0 4.87 90) (layer "F.Fab")
+    (fp_text value "CVBS" (at 0 4.87 90) (layer "F.Fab")
         (effects (font (size 1 1) (thickness 0.15)))
     )
@@
         (effects (font (size 1 1) (thickness 0.15)))
     )
-    (fp_text value "6.8Ω" (at 0 2.28 90) (layer "F.Fab")
+    (fp_text value "0.68Ω" (at 0 2.28 90) (layer "F.Fab")
         (effects (font (size 1 1) (thickness 0.15)))
     )
@@
   (segment (start 191 83.75) (end 186 83.75) (width 0.25) (layer "F.Cu") (net 40))
   (segment (start 196.5 120) (end 197 120) (width 0.25) (layer "F.Cu") (net 40))
+  (segment (start 139.655 76.85) (end 139.655 79.5) (width 0.25) (layer "F.Cu") (net 40))
   (segment (start 179.084999 123.084999) (end 181.25 125.25) (width 0.25) (layer "F.Cu") (net 40))
   (segment (start 175.25 61.25) (end 178.035715 61.25) (width 0.25) (layer "F.Cu") (net 40))
@@
   (segment (start 161.5675 72.3175) (end 161.5 72.25) (width 0.25) (layer "F.Cu") (net 40))
   (segment (start 182.75 114.3175) (end 182.75 114.5) (width 0.25) (layer "F.Cu") (net 40))
+  (segment (start 139.655 79.5) (end 137.75 79.5) (width 0.25) (layer "F.Cu") (net 40))
   (segment (start 188.75 96.3175) (end 188.8175 96.3175) (width 0.25) (layer "F.Cu") (net 40))
   (segment (start 161.4325 71.1825) (end 161.5 71.25) (width 0.25) (layer "F.Cu") (net 40))

Commit message: Use only the positive outputs of PAM8003 (as a unipolar amplifier), because negative outputs can't be tied together.
Parts:
- removed JP5: Common Negative Jumper, Jumper:SolderJumper-2_P1.3mm_Bridged2Bar_RoundedPad1.0x1.5mm
- L6: value 6.8uH -> 22uH
- U10: value 25x128 -> 25x40
- U9: value 24x01 -> 24x04
Connections:
- J13 pad R2: LEFT- -> unconnected-(J13-PadR2)
- J13 pad S: RIGHT- -> GND
- U7 pad 15: RIGHT- -> unconnected-(U7-ROUT--Pad15)
- U7 pad 2: LEFT- -> unconnected-(U7-LOUT--Pad2)
Routing:
- net LEFT-: track 21.8 -> 0.00 mm, vias 2 -> 0
- net RIGHT-: track 17.5 -> 0.00 mm, vias 2 -> 0
